File: Switchless-Addon-1chip/SNES_AddOn1Chip.brd (EAGLE design)
At the start: 29.2 x 25.9 mm, 19 parts, among them X50 17.734M, X60 21.477M

Commit message: Just a few Updates
Changed lines of the file:
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@@
 <contactref element="C2" pad="2"/>
 <contactref element="PAD5" pad="1"/>
-<via x="21.59" y="24.765" extent="1-16" drill="0.6"/>
-<via x="24.13" y="21.59" extent="1-16" drill="0.6"/>
+<via x="21.59" y="23.8125" extent="1-16" drill="0.6"/>
+<via x="24.13" y="25.0825" extent="1-16" drill="0.6"/>
 <via x="30.48" y="34.29" extent="1-16" drill="0.6"/>
 <via x="28.575" y="38.1" extent="1-16" drill="0.6"/>
@@
 </polygon>
 <via x="20.32" y="42.8625" extent="1-16" drill="0.6"/>
+<via x="24.13" y="23.8125" extent="1-16" drill="0.6"/>
+<via x="21.59" y="25.0825" extent="1-16" drill="0.6"/>
+<via x="22.86" y="23.8125" extent="1-16" drill="0.6"/>
+<via x="22.86" y="25.0825" extent="1-16" drill="0.6"/>
 </signal>
 <signal name="VCC">
