File: digAudio/digAudio.brd (EAGLE design)
At the start: 18.4 x 37.5 mm, 12 parts

Commit message: Just a few Updates
Parts:
- moved GND 15.2 mm to (8.89, 7.62)
- moved VCC 15.2 mm to (24.1, 7.62)
Routing:
- net VCC: track 53.2 -> 41.7 mm, vias 7 -> 11
- net N$3: track 12.3 -> 10.9 mm, vias 0 -> 2
- net N$2: track 14.8 -> 13.4 mm, vias 0 -> 2
- net N$6: track 14.3 -> 15.0 mm, vias 0 -> 2
- added copper zone on layer 16, net GND
- added copper zone on layer 1, net VCC
