File: RGB_Amp_Mini/SNES_RGBAmp.sch (EAGLE design)
At the start: 10 parts

Commit message: Replace unused solder points at the MultiAV by simple holes
Parts:
- removed U$2: SNES_MULTIAV, snescart:SNES_MULTIAV
- added U$3: SNES_MULTIAV_RGBC_ONLY, snes_div:SNES_MULTIAV_RGBC_ONLY
Connections:
- net GND: now also U$3G$2.GND, U$3G$3.GND; no longer U$2G$2.GND, U$2G$3.GND
- net N$10: now also U$3G$1./CS; no longer U$2G$1./CS
- net N$5: now also U$3G$1.RED; no longer U$2G$1.RED
- net N$6: now also U$3G$1.GREEN; no longer U$2G$1.GREEN
- net N$9: now also U$3G$1.BLUE; no longer U$2G$1.BLUE
- net VCC: now also U$3G$3.VCC; no longer U$2G$2.VCC
Changed lines of the file:
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@@
 <?xml version="1.0" encoding="utf-8"?>
 <!DOCTYPE eagle SYSTEM "eagle.dtd">
-<eagle version="6.5.0">
+<eagle version="7.0.0">
 <drawing>
 <settings>
@@
 <parts>
 <part name="U$1" library="snescart" deviceset="THS7314" device=""/>
-<part name="U$2" library="snescart" deviceset="SNES_MULTIAV" device=""/>
 <part name="R2" library="snescart" deviceset="R0805" device="" value="100"/>
 <part name="R3" library="snescart" deviceset="R0805" device="" value="100"/>
@@
 <part name="B" library="wirepad" deviceset="SMD2" device=""/>
 <part name="CS" library="wirepad" deviceset="SMD2" device=""/>
+<part name="U$3" library="snes_div" deviceset="SNES_MULTIAV_RGBC_ONLY" device=""/>
 </parts>
 <sheets>
@@
 <instances>
 <instance part="U$1" gate="G$1" x="0" y="-2.54"/>
-<instance part="U$2" gate="G$1" x="53.34" y="-15.24"/>
 <instance part="R2" gate="G$1" x="25.4" y="0"/>
 <instance part="R3" gate="G$1" x="25.4" y="-7.62"/>
 <instance part="R1" gate="G$1" x="25.4" y="-15.24"/>
 <instance part="U$1" gate="G$2" x="-12.7" y="-20.32" rot="R90"/>
-<instance part="U$2" gate="G$2" x="-12.7" y="-22.86" rot="R90"/>
-<instance part="U$2" gate="G$3" x="-5.08" y="-25.4" rot="R90"/>
 <instance part="P+1" gate="VCC" x="-25.4" y="-10.16"/>
 <instance part="GND1" gate="1" x="0" y="-30.48"/>
@@
 <instance part="B" gate="1" x="-25.4" y="-5.08"/>
 <instance part="CS" gate="1" x="15.24" y="-22.86"/>
+<instance part="U$3" gate="G$1" x="53.34" y="-2.54"/>
+<instance part="U$3" gate="G$2" x="-5.08" y="-25.4" rot="R90"/>
+<instance part="U$3" gate="G$3" x="-12.7" y="-22.86" rot="R90"/>
 </instances>
 <busses>
@@
 <pinref part="R3" gate="G$1" pin="2"/>
 <wire x1="33.02" y1="-7.62" x2="30.48" y2="-7.62" width="0.1524" layer="91"/>
-<pinref part="U$2" gate="G$1" pin="GREEN"/>
 <wire x1="43.18" y1="-2.54" x2="33.02" y2="-2.54" width="0.1524" layer="91"/>
+<pinref part="U$3" gate="G$1" pin="GREEN"/>
 </segment>
 </net>
@@
 <wire x1="30.48" y1="-15.24" x2="35.56" y2="-15.24" width="0.1524" layer="91"/>
 <wire x1="35.56" y1="-15.24" x2="35.56" y2="-5.08" width="0.1524" layer="91"/>
-<pinref part="U$2" gate="G$1" pin="BLUE"/>
 <wire x1="35.56" y1="-5.08" x2="43.18" y2="-5.08" width="0.1524" layer="91"/>
+<pinref part="U$3" gate="G$1" pin="BLUE"/>
 </segment>
 </net>
@@
 <segment>
 <pinref part="GND1" gate="1" pin="GND"/>
-<pinref part="U$2" gate="G$3" pin="GND"/>
 <wire x1="0" y1="-27.94" x2="0" y2="-25.4" width="0.1524" layer="91"/>
-<pinref part="U$2" gate="G$2" pin="GND"/>
-<wire x1="0" y1="-25.4" x2="0" y2="-22.86" width="0.1524" layer="91"/>
-<junction x="0" y="-25.4"/>
+<pinref part="U$3" gate="G$2" pin="GND"/>
 <pinref part="U$1" gate="G$2" pin="GND"/>
-<wire x1="0" y1="-22.86" x2="0" y2="-20.32" width="0.1524" layer="91"/>
-<junction x="0" y="-22.86"/>
 <pinref part="C1" gate="G$1" pin="2"/>
 <wire x1="-7.62" y1="-15.24" x2="0" y2="-15.24" width="0.1524" layer="91"/>
 <wire x1="0" y1="-15.24" x2="0" y2="-20.32" width="0.1524" layer="91"/>
+<pinref part="U$3" gate="G$3" pin="GND"/>
+<wire x1="0" y1="-22.86" x2="0" y2="-20.32" width="0.1524" layer="91"/>
 <junction x="0" y="-20.32"/>
+<wire x1="0" y1="-25.4" x2="0" y2="-22.86" width="0.1524" layer="91"/>
+<junction x="0" y="-25.4"/>
+<junction x="0" y="-22.86"/>
 </segment>
 </net>
 <net name="VCC" class="0">
 <segment>
-<pinref part="U$2" gate="G$2" pin="VCC"/>
 <pinref part="U$1" gate="G$2" pin="VCC"/>
-<wire x1="-25.4" y1="-22.86" x2="-25.4" y2="-20.32" width="0.1524" layer="91"/>
 <pinref part="P+1" gate="VCC" pin="VCC"/>
 <wire x1="-25.4" y1="-12.7" x2="-25.4" y2="-15.24" width="0.1524" layer="91"/>
-<junction x="-25.4" y="-20.32"/>
 <pinref part="C1" gate="G$1" pin="1"/>
 <wire x1="-25.4" y1="-15.24" x2="-25.4" y2="-20.32" width="0.1524" layer="91"/>
 <wire x1="-15.24" y1="-15.24" x2="-25.4" y2="-15.24" width="0.1524" layer="91"/>
 <junction x="-25.4" y="-15.24"/>
+<pinref part="U$3" gate="G$3" pin="VCC"/>
+<wire x1="-25.4" y1="-20.32" x2="-25.4" y2="-22.86" width="0.1524" layer="91"/>
+<junction x="-25.4" y="-20.32"/>
 </segment>
 </net>
@@
 <segment>
 <pinref part="R2" gate="G$1" pin="2"/>
-<pinref part="U$2" gate="G$1" pin="RED"/>
 <wire x1="43.18" y1="0" x2="30.48" y2="0" width="0.1524" layer="91"/>
+<pinref part="U$3" gate="G$1" pin="RED"/>
 </segment>
 </net>
@@
 <wire x1="17.78" y1="-22.86" x2="38.1" y2="-22.86" width="0.1524" layer="91"/>
 <wire x1="38.1" y1="-22.86" x2="38.1" y2="-7.62" width="0.1524" layer="91"/>
-<pinref part="U$2" gate="G$1" pin="/CS"/>
 <wire x1="38.1" y1="-7.62" x2="43.18" y2="-7.62" width="0.1524" layer="91"/>
-</segment>
-</net>
+<pinref part="U$3" gate="G$1" pin="/CS"/>
+</segment>
+</net>
