File: RGB_Amp_Mini/SNES_RGBAmp.brd (EAGLE design)
At the start: 18.4 x 17.8 mm, 10 parts

Commit message: Replace unused solder points at the MultiAV by simple holes
Parts:
- removed U$2: SNES_MULTIAV, snescart:SNES_MULTIAV
- added U$3: SNES_MULTIAV_RGBC_ONLY, snes_div:SNES_MULTIAV_RGBC_ONLY
Connections:
- net GND: now also U$3.P$5, U$3.P$6; no longer U$2.P$5, U$2.P$6
- net N$10: now also U$3.P$3; no longer U$2.P$3
- net N$5: now also U$3.P$1; no longer U$2.P$1
- net N$6: now also U$3.P$2; no longer U$2.P$2
- net N$9: now also U$3.P$4; no longer U$2.P$4
- net VCC: now also U$3.P$10; no longer U$2.P$10
Changed lines of the file:
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@@
 <?xml version="1.0" encoding="utf-8"?>
 <!DOCTYPE eagle SYSTEM "eagle.dtd">
-<eagle version="6.5.0">
+<eagle version="7.0.0">
 <drawing>
 <settings>
@@
 <pass name="Default">
 <param name="RoutingGrid" value="50mil"/>
+<param name="AutoGrid" value="1"/>
+<param name="Efforts" value="0"/>
+<param name="TopRouterVariant" value="1"/>
 <param name="tpViaShape" value="round"/>
 <param name="PrefDir.1" value="|"/>
@@
 <elements>
 <element name="U$1" library="snescart" package="THS7314" value="THS7314" x="12.7" y="8.41375" smashed="yes" rot="R90"/>
-<element name="U$2" library="snescart" package="SNES_MULTIAV" value="SNES_MULTIAV" x="10.16" y="18.415"/>
 <element name="R2" library="snescart" package="Z0805" value="100" x="19.05" y="13.6525" smashed="yes" rot="R90"/>
 <element name="R3" library="snescart" package="Z0805" value="100" x="19.05" y="18.57375" smashed="yes" rot="R90"/>
@@
 <attribute name="NAME" x="18.11625" y="4.915" size="1.016" layer="25" font="vector" ratio="12" rot="R180"/>
 </element>
+<element name="U$3" library="snes_div" package="SNES_MULTIAV_RGBC_ONLY" value="SNES_MULTIAV_RGBC_ONLY" x="10.16" y="18.415"/>
 </elements>
 <signals>
@@
 <signal name="N$6">
 <contactref element="R3" pad="2"/>
-<contactref element="U$2" pad="P$2"/>
-<wire x1="16.51" y1="19.685" x2="19.05" y2="19.685" width="0.3048" layer="1"/>
 <wire x1="19.05" y1="19.685" x2="19.05" y2="19.52375" width="0.3048" layer="1"/>
+<contactref element="U$3" pad="P$2"/>
+<wire x1="16.51" y1="19.685" x2="18.88875" y2="19.685" width="0.3048" layer="1"/>
+<wire x1="18.88875" y1="19.685" x2="19.05" y2="19.52375" width="0.3048" layer="1"/>
 </signal>
 <signal name="N$7">
@@
 <signal name="N$9">
 <contactref element="R1" pad="2"/>
-<contactref element="U$2" pad="P$4"/>
 <wire x1="16.51" y1="14.6025" x2="16.51" y2="14.605" width="0.3048" layer="1"/>
 <wire x1="16.51" y1="14.605" x2="15.24" y2="15.875" width="0.3048" layer="1"/>
 <wire x1="15.24" y1="15.875" x2="15.24" y2="18.415" width="0.3048" layer="1"/>
-<wire x1="15.24" y1="18.415" x2="13.97" y2="19.685" width="0.3048" layer="1"/>
+<contactref element="U$3" pad="P$4"/>
+<wire x1="13.97" y1="19.685" x2="15.24" y2="18.415" width="0.3048" layer="1"/>
 </signal>
 <signal name="GND">
-<contactref element="U$2" pad="P$6"/>
-<contactref element="U$2" pad="P$5"/>
-<contactref element="U$1" pad="5"/>
-<contactref element="C1" pad="2"/>
 <polygon width="0.254" layer="1">
 <vertex x="0" y="0"/>
@@
 <via x="8.89" y="11.43" extent="1-16" drill="0.6"/>
 <via x="15.24" y="4.7625" extent="1-16" drill="0.6"/>
+<contactref element="U$3" pad="P$5"/>
+<contactref element="U$1" pad="5"/>
+<contactref element="C1" pad="2"/>
+<contactref element="U$3" pad="P$6"/>
 </signal>
 <signal name="VCC">
-<contactref element="U$2" pad="P$10"/>
 <contactref element="U$1" pad="4"/>
 <contactref element="C1" pad="1"/>
@@
 <wire x1="10.16" y1="17.78" x2="9.525" y2="18.415" width="0.3048" layer="1"/>
 <wire x1="9.525" y1="18.415" x2="7.62" y2="18.415" width="0.3048" layer="1"/>
-<wire x1="7.62" y1="18.415" x2="6.35" y2="19.685" width="0.3048" layer="1"/>
 <wire x1="9.525" y1="13.335" x2="9.525" y2="15.24" width="0.3048" layer="1"/>
 <wire x1="9.525" y1="15.24" x2="10.16" y2="15.875" width="0.3048" layer="1"/>
 <wire x1="10.16" y1="15.875" x2="10.16" y2="17.78" width="0.3048" layer="1"/>
+<contactref element="U$3" pad="P$10"/>
+<wire x1="7.62" y1="18.415" x2="6.35" y2="19.685" width="0.3048" layer="1"/>
 </signal>
 <signal name="N$5">
 <contactref element="R2" pad="2"/>
-<contactref element="U$2" pad="P$1"/>
+<contactref element="U$3" pad="P$1"/>
 <wire x1="16.51" y1="17.145" x2="16.51" y2="17.1425" width="0.3048" layer="1"/>
 <wire x1="16.51" y1="17.1425" x2="19.05" y2="14.6025" width="0.3048" layer="1"/>
@@
 <signal name="N$10">
 <contactref element="CS" pad="1"/>
-<contactref element="U$2" pad="P$3"/>
 <via x="13.97" y="8.89" extent="1-16" drill="0.6"/>
 <wire x1="19.3675" y1="4.445" x2="17.78" y2="4.445" width="0.3048" layer="1"/>
@@
 <wire x1="15.24" y1="10.16" x2="15.24" y2="12.7" width="0.3048" layer="16"/>
 <wire x1="15.24" y1="12.7" x2="13.97" y2="13.97" width="0.3048" layer="16"/>
-<wire x1="13.97" y1="13.97" x2="13.97" y2="17.145" width="0.3048" layer="16"/>
+<contactref element="U$3" pad="P$3"/>
+<wire x1="13.97" y1="17.145" x2="13.97" y2="13.97" width="0.3048" layer="16"/>
 </signal>
 </signals>

Commit message: Update silkscreen
Routing:
- net N$10: track 18.0 -> 18.8 mm
Other:
- board text added: "RGBAmp V2.1m SNES mini/jr. by borti4938"
- board text added: "THS 7314"
- board text added: "__/)__/)_"
- board text added: "borti4938"
- board text removed: "1"
- board text removed: "SNES-Mini"
- board text removed: "THS7314"
Changed lines of the file:
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@@
 <?xml version="1.0" encoding="utf-8"?>
 <!DOCTYPE eagle SYSTEM "eagle.dtd">
-<eagle version="7.0.0">
+<eagle version="6.5.0">
 <drawing>
 <settings>
@@
 <board>
 <plain>
-<text x="8.54075" y="4.60375" size="1.016" layer="21" font="vector" ratio="12">THS7314</text>
+<text x="13.97" y="6.6675" size="0.8128" layer="21" font="vector" ratio="15" rot="R90"> THS
+7314</text>
 <text x="15.24" y="11.90625" size="1.016" layer="25" font="vector" ratio="12" rot="R90">R1
 R2|R3</text>
@@
 <wire x1="20.32" y1="20.955" x2="3.81" y2="20.955" width="0" layer="20"/>
 <wire x1="2.54" y1="19.685" x2="2.54" y2="16.98625" width="0" layer="20"/>
-<text x="13.49375" y="6.35" size="1.016" layer="25" font="vector" ratio="12">1</text>
 <wire x1="3.81" y1="15.875" x2="2.54" y2="16.98625" width="0" layer="20" curve="-82.371791"/>
 <wire x1="3.81" y1="20.955" x2="2.54" y2="19.685" width="0" layer="20" curve="90"/>
 <wire x1="13.97" y1="11.90625" x2="13.97" y2="15.71625" width="0.127" layer="25"/>
 <wire x1="12.7" y1="13.840734375" x2="15.24" y2="13.840734375" width="0.127" layer="25"/>
-<text x="8.54075" y="3.33375" size="1.016" layer="21" font="vector" ratio="12">SNES-Mini</text>
+<text x="8.6995" y="4.60375" size="1.016" layer="21" font="vector" ratio="12">borti4938</text>
 <wire x1="16.35125" y1="5.08" x2="17.78" y2="5.08" width="0.12191875" layer="25"/>
+<text x="8.85825" y="3.4925" size="0.8128" layer="21" font="vector" ratio="15">__/)__/)_</text>
+<text x="19.84375" y="11.27125" size="1.016" layer="22" rot="MR0">RGBAmp V2.1m
+SNES mini/jr.
+by borti4938</text>
 </plain>
 <attributes>
@@
 <pass name="Default">
 <param name="RoutingGrid" value="50mil"/>
-<param name="AutoGrid" value="1"/>
-<param name="Efforts" value="0"/>
-<param name="TopRouterVariant" value="1"/>
 <param name="tpViaShape" value="round"/>
 <param name="PrefDir.1" value="|"/>
@@
 </signal>
 <signal name="GND">
-<polygon width="0.254" layer="1">
+<polygon width="0.254" layer="1" thermals="no">
 <vertex x="0" y="0"/>
 <vertex x="24.13" y="0"/>
@@
 <vertex x="0" y="22.86"/>
 </polygon>
-<polygon width="0.254" layer="16">
+<polygon width="0.254" layer="16" thermals="no">
 <vertex x="0" y="22.86"/>
 <vertex x="24.13" y="22.86"/>
@@
 </polygon>
 <via x="8.89" y="11.43" extent="1-16" drill="0.6"/>
-<via x="15.24" y="4.7625" extent="1-16" drill="0.6"/>
+<via x="12.7" y="4.1275" extent="1-16" drill="0.6"/>
 <contactref element="U$3" pad="P$5"/>
 <contactref element="U$1" pad="5"/>
@@
 <signal name="N$10">
 <contactref element="CS" pad="1"/>
+<contactref element="U$3" pad="P$3"/>
+<wire x1="19.3675" y1="4.445" x2="14.605" y2="4.445" width="0.3048" layer="1"/>
+<wire x1="14.605" y1="4.445" x2="13.97" y2="5.08" width="0.3048" layer="1"/>
+<wire x1="13.97" y1="5.08" x2="13.97" y2="8.89" width="0.3048" layer="1"/>
 <via x="13.97" y="8.89" extent="1-16" drill="0.6"/>
-<wire x1="19.3675" y1="4.445" x2="17.78" y2="4.445" width="0.3048" layer="1"/>
-<wire x1="17.78" y1="4.445" x2="16.51" y2="5.715" width="0.3048" layer="1"/>
-<wire x1="16.51" y1="5.715" x2="14.605" y2="5.715" width="0.3048" layer="1"/>
-<wire x1="14.605" y1="5.715" x2="13.97" y2="6.35" width="0.3048" layer="1"/>
-<wire x1="13.97" y1="6.35" x2="13.97" y2="8.89" width="0.3048" layer="1"/>
 <wire x1="13.97" y1="8.89" x2="15.24" y2="10.16" width="0.3048" layer="16"/>
 <wire x1="15.24" y1="10.16" x2="15.24" y2="12.7" width="0.3048" layer="16"/>
 <wire x1="15.24" y1="12.7" x2="13.97" y2="13.97" width="0.3048" layer="16"/>
-<contactref element="U$3" pad="P$3"/>
-<wire x1="13.97" y1="17.145" x2="13.97" y2="13.97" width="0.3048" layer="16"/>
+<wire x1="13.97" y1="13.97" x2="13.97" y2="17.145" width="0.3048" layer="16"/>
 </signal>
 </signals>
