File: Switchless-1Chip-all/SNES1Chip_SCIC_IGR_D4_Takt_SMD.brd (EAGLE design)
At the start: 60.3 x 35.9 mm, 47 parts

Commit message: Update
Parts:
- removed J1-L_TYPE: (no value), jumper:JP2
- removed LED-OUT: (no value), pinhead:1X02
- removed NTSC:21.477MHZ, PAL:17.734MHZ: (no value), crystal:HC49/S
- added NTSC_21.477MHZ, PAL_17.734MHZ: MY_CRYSTALS, snes_div:MY_SMD_CRYSTAL2
- added PAD3, PAD4: (no value), wirepad:SMD1,27-2,54
- added U$1, U$2: MY_JUMPER, snes_div:MYJUMP
- +5V, /PARD, D4, GND, MODE, P0, P1, P2, P3, P4, P5, P6, P7, PAD1, PAD10, PAD11, PAD2, PAD7, PAD8, PIN2, PIN3, PIN4, PIN9, RIGHT: device wirepad:2,54/0,8 -> wirepad:SMD1,27-2,54
- UIGR: value uIGR -> uIGR(V2)
- moved C2 0.95 mm to (37.8, 4.13)
- moved C3 0.95 mm to (54.9, 4.13)
- moved C4 0.95 mm to (37.8, 27.6)
- moved C5 0.95 mm to (54.9, 27.6)
Connections:
- net +5V: now also U$2.P$1; no longer J1-L_TYPE.1
- net GND: now also U$1.P$2; no longer J1-L_TYPE.3
- net N$14: now also PAD4.1; no longer LED-OUT.2
- net N$27: now also PAL_17.734MHZ.1; no longer PAL:17.734MHZ.1
- net N$28: now also PAL_17.734MHZ.2; no longer PAL:17.734MHZ.2
- net N$29: now also NTSC_21.477MHZ.1; no longer NTSC:21.477MHZ.1
- net N$30: now also NTSC_21.477MHZ.2; no longer NTSC:21.477MHZ.2
- net N$5: now also PAD3.1; no longer LED-OUT.1
- net N$8: now also U$1.P$1, U$2.P$2; no longer J1-L_TYPE.2
Routing:
- net +5V: track 133.7 -> 139.4 mm, vias 7 -> 8
- net N$12: track 8.72 -> 12.9 mm, vias 1 -> 0
- net N$33: track 56.7 -> 52.6 mm
- net N$8: track 21.2 -> 24.3 mm, vias 1 -> 2
- net N$34: track 35.4 -> 32.9 mm
- net N$18: track 9.35 -> 10.8 mm, vias 1 -> 2
- net N$42: track 32.9 -> 31.7 mm, vias 2 -> 4
- net N$5: track 37.1 -> 38.1 mm, vias 1 -> 2
- net N$29: track 14.9 -> 14.3 mm
- net N$27: track 15.9 -> 15.4 mm
- net N$30: track 18.5 -> 19.0 mm
- net N$28: track 18.2 -> 18.7 mm
- net N$3: track 27.9 -> 27.5 mm, vias 1 -> 2
- net GND: vias 16 -> 20
- net N$14: vias 1 -> 2
Other:
- board text added: "(16F684)"
- board text added: "12"
- board text added: "17.734MHz"
- board text added: "21.477MHz"
- board text added: "23"
- board text added: "74HC(T) 125"
- board text added: ": S-PPU1 Pin24 | S-PPU2 Pin30 : S-CPUN Pin111"
- board text added: "= solder to Pin = solder to Pad = Pin lifted"
- board text added: "LED-Colors"
- board text added: "Mode-Output to SNES 2Chip 1Chip"
- board text added: "NTSC"
- board text added: "NTSC-Crystal:"
- board text added: "PAL"
- board text added: "PAL-Crystal:"
- board text added: "PIC16F630"
- board text added: "PIN PAD (Pl)"
- board text added: "PPU:"
- board text added: "Parts for 1Chip-SNES"
- board text added: "X1(ri)"
- board text removed: "(Pl, R2)"
- board text removed: "(R2)"
- board text removed: "2xPIC16F630"
- board text removed: ": PPU1 Pin24 | PPU2 Pin30 : S-CPUN Pin 111"
- board text removed: "= solder to Pin = solder to Pad = Pin lifted = for SNES Rev.2 only"
- board text removed: "LED-Colors for"
- board text removed: "Mode-Output to SNES 1st Revi. 2nd Revi."
- board text removed: "NTSC | PAL"
- board text removed: "NTSC-Crystal: 21.477MHz"
- board text removed: "PAL-Crystal: 17.734MHz"
- board text removed: "PIN PAD (Pl) (R2)"
- board text removed: "PPU(s):"
- board text removed: "X1 (R2) (right)"
