File: Switchless-1Chip-all/SNES1Chip_SCIC_IGR_D4_Takt_SMD.sch (EAGLE design)
At the start: 47 parts

Commit message: Update
Parts:
- removed J1-L_TYPE: (no value), jumper:JP2E
- removed LED-OUT: (no value), pinhead:PINHD-1X2
- removed NTSC:21.477MHZ, PAL:17.734MHZ: (no value), crystal:CRYSTALHC49S
- added NTSC_21.477MHZ, PAL_17.734MHZ: MY_CRYSTALS, snes_div:MY_CRYSTALS
- added PAD3, PAD4: (no value), wirepad:SMD2
- added U$1, U$2: MY_JUMPER, snes_div:MY_JUMPER
- +5V, /PARD, D4, GND, MODE, P0, P1, P2, P3, P4, P5, P6, P7, PAD1, PAD10, PAD11, PAD2, PAD7, PAD8, PIN2, PIN3, PIN4, PIN9, RIGHT: device wirepad:2,54/0,8 -> wirepad:SMD2
- UIGR: value uIGR -> uIGR(V2)
Connections:
- net +5V: now also U$2.1; no longer J1-L_TYPE.1
- net GND: now also U$1.2; no longer J1-L_TYPE.3
- net N$14: now also PAD4.P; no longer LED-OUT.2
- net N$27: now also PAL_17.734MHZ.1; no longer PAL:17.734MHZ.1
- net N$28: now also PAL_17.734MHZ.2; no longer PAL:17.734MHZ.2
- net N$29: now also NTSC_21.477MHZ.1; no longer NTSC:21.477MHZ.1
- net N$30: now also NTSC_21.477MHZ.2; no longer NTSC:21.477MHZ.2
- net N$5: now also PAD3.P; no longer LED-OUT.1
- net N$8: now also U$1.1, U$2.2; no longer J1-L_TYPE.2
